File: tester_remotos/tester_remotos.sch (KiCad schematic (older format))
At the start: 15 parts, among them J1 USB_B, Q1 BC548, U1 4093, U2 VS1838B

Commit message: Módulo "probador de control remoto" terminado.
Parts:
- added J2, J3: CONN_01X01, Wire_Pads:SolderWirePad_single_1mmDrill, symbol CONN_01X01
- U2: footprint Pin_Headers:Pin_Header_Straight_1x03 -> opto:VS1838B
Connections:
- net +5V: now also J2.1 (P1)
- net GND: now also J3.1 (P1)
Other:
- moved on the sheet: C1
Changed lines of the file:
@@
 	5575 5625 5575 5800
 Wire Wire Line
-	6200 5025 5575 5025
+	5575 5025 6200 5025
 Connection ~ 5575 5025
 Wire Wire Line
@@
 L +5V #PWR011
 U 1 1 5AEE20B0
-P 2400 1100
-F 0 "#PWR011" H 2400 950 50  0001 C CNN
-F 1 "+5V" H 2400 1240 50  0000 C CNN
-F 2 "" H 2400 1100 60  0000 C CNN
-F 3 "" H 2400 1100 60  0000 C CNN
-	1    2400 1100
-	1    0    0    -1
-$EndComp
-Wire Wire Line
-	2400 1100 2400 1350
+P 2625 1100
+F 0 "#PWR011" H 2625 950 50  0001 C CNN
+F 1 "+5V" H 2625 1240 50  0000 C CNN
+F 2 "" H 2625 1100 60  0000 C CNN
+F 3 "" H 2625 1100 60  0000 C CNN
+	1    2625 1100
+	1    0    0    -1
+$EndComp
+Wire Wire Line
+	2625 1100 2625 1350
 $Comp
 L GND #PWR012
@@
 L C C1
 U 1 1 5AEE2708
-P 2400 1500
-F 0 "C1" H 2425 1600 50  0000 L CNN
-F 1 "100nf" H 2425 1400 50  0000 L CNN
-F 2 "Capacitors_ThroughHole:C_Disc_D6_P5" H 2438 1350 50  0001 C CNN
-F 3 "" H 2400 1500 50  0001 C CNN
-	1    2400 1500
-	1    0    0    -1
-$EndComp
-Connection ~ 2400 1225
+P 2625 1500
+F 0 "C1" H 2650 1600 50  0000 L CNN
+F 1 "100nf" H 2650 1400 50  0000 L CNN
+F 2 "Capacitors_ThroughHole:C_Disc_D6_P5" H 2663 1350 50  0001 C CNN
+F 3 "" H 2625 1500 50  0001 C CNN
+	1    2625 1500
+	1    0    0    -1
+$EndComp
+Connection ~ 2625 1225
 $Comp
 L GND #PWR013
 U 1 1 5AEE27BE
-P 2400 1700
-F 0 "#PWR013" H 2400 1450 50  0001 C CNN
-F 1 "GND" H 2400 1550 50  0000 C CNN
-F 2 "" H 2400 1700 60  0000 C CNN
-F 3 "" H 2400 1700 60  0000 C CNN
-	1    2400 1700
-	1    0    0    -1
-$EndComp
-Wire Wire Line
-	2400 1650 2400 1700
+P 2625 1700
+F 0 "#PWR013" H 2625 1450 50  0001 C CNN
+F 1 "GND" H 2625 1550 50  0000 C CNN
+F 2 "" H 2625 1700 60  0000 C CNN
+F 3 "" H 2625 1700 60  0000 C CNN
+	1    2625 1700
+	1    0    0    -1
+$EndComp
+Wire Wire Line
+	2625 1650 2625 1700
 $Comp
 L VS1838B U2
@@
 F 0 "U2" H 1500 3750 50  0000 L CNN
 F 1 "VS1838B" H 1500 3150 50  0000 L CNN
-F 2 "Pin_Headers:Pin_Header_Straight_1x03" H 1850 3075 50  0001 C CNN
+F 2 "opto:VS1838B" H 1850 3075 50  0001 C CNN
 F 3 "" H 2550 3750 50  0000 C CNN
 	1    1900 3450
@@
 $EndComp
 Wire Wire Line
-	1550 2050 1650 2050
-Wire Wire Line
-	1950 1225 2400 1225
+	1550 2050 2250 2050
+Wire Wire Line
+	1950 1225 2625 1225
+$Comp
+L CONN_01X01 J2
+U 1 1 5AF72734
+P 2250 900
+F 0 "J2" H 2250 1000 50  0000 C CNN
+F 1 "CONN_01X01" V 2350 900 50  0000 C CNN
+F 2 "Wire_Pads:SolderWirePad_single_1mmDrill" H 2250 900 50  0001 C CNN
+F 3 "" H 2250 900 50  0001 C CNN
+	1    2250 900
+	0    -1   -1   0
+$EndComp
+$Comp
+L CONN_01X01 J3
+U 1 1 5AF72A67
+P 2250 1725
+F 0 "J3" H 2250 1825 50  0000 C CNN
+F 1 "CONN_01X01" V 2350 1725 50  0000 C CNN
+F 2 "Wire_Pads:SolderWirePad_single_1mmDrill" H 2250 1725 50  0001 C CNN
+F 3 "" H 2250 1725 50  0001 C CNN
+	1    2250 1725
+	0    -1   -1   0
+$EndComp
+Wire Wire Line
+	2250 2050 2250 1925
+Wire Wire Line
+	2250 1100 2250 1225
+Connection ~ 2250 1225
 $EndSCHEMATC

Commit message: Modificado de pads de varios footprints. Correción de algunos textos en esquemático.
Other:
- note added: "C1 es thru-hole. C2 es SMD.\nUsar cualquiera de los 2.\nVR1 cambia con la elección del capacitor:\n1uf -> 2.2K\n100nf -> 22K"
- note removed: "C1 es truehole. C2 es SMD.\nUsar cualquiera de los 2.\nVR1 cambia con la elección del capacitor:\n1uf -> 2.2K\n100nf -> 22K"
Changed lines of the file:
@@
 Connection ~ 5575 5675
 Text Notes 6650 5875 0    60   ~ 0
-C1 es truehole.  C2 es SMD.\nUsar cualquiera de los 2.\nVR1 cambia con la elección del capacitor:\n1uf -> 2.2K\n100nf -> 22K
+C1 es thru-hole.  C2 es SMD.\nUsar cualquiera de los 2.\nVR1 cambia con la elección del capacitor:\n1uf -> 2.2K\n100nf -> 22K
 $Comp
 L +5V #PWR011
